Commit message: upgrade to latest genesis world release. prepared go2w training.

File: ressources/robots/go2w/urdf/go2w_description.urdf (robot description, URDF)
Before this commit: robot go2w_description, 40 links, 39 joints
Links:
- link FL_foot: geometry collision cylinder length=0.052 radius=0.086; visual mesh filename=../dae/left_wheel.dae
- link FR_foot: geometry collision cylinder length=0.052 radius=0.086; visual mesh filename=../dae/right_wheel.dae
- link RL_foot: geometry collision cylinder length=0.052 radius=0.086; visual mesh filename=../dae/left_wheel.dae
- link RR_foot: geometry collision cylinder length=0.052 radius=0.086; visual mesh filename=../dae/right_wheel.dae

Commit message: added mass/inertia of realsense camera to urdf.

File: ressources/robots/go2w/urdf/go2w_description.urdf (robot description, URDF)
Before this commit: robot go2w_description, 40 links, 39 joints
Links:
- link front_realsense_body: mass 0 -> 0.11598
